File: mainboard/mainboard.kicad_sch (KiCad schematic)
At the start: 68 parts, among them J1 Eurorack_Power, Q1 2N3906, Q2 2N3906, Q3 2N3904, Q4 2N3904, U1 40106, U2 TL074, U4 4070, U5 4520, U6 4015, U7 4015

Commit message: Routing done, panel done
Parts:
- J2: value (none) -> Osc1_Socket; footprint (none) -> Connector_PinSocket_2.54mm:PinSocket_1x12_P2.54mm_Vertical
- J3: value (none) -> Osc2_Socket; footprint (none) -> Connector_PinSocket_2.54mm:PinSocket_1x12_P2.54mm_Vertical
Connections:
- net Clk2: now also J3.7 (Pin_7); no longer J3.8 (Pin_8)
- net D1: now also J2.5 (Pin_5); no longer J2.4 (Pin_4)
- net O1: now also U1.10; no longer U1.4
- net O2: now also U1.4; no longer U1.10
- net Osc1: now also J2.6 (Pin_6), U4.2; no longer J2.7 (Pin_7), U4.1
- net Osc2: now also J3.5 (Pin_5), U4.1; no longer J3.7 (Pin_7), U4.2
- net Osc3sw: now also J3.3 (Pin_3); no longer J3.5 (Pin_5)
- net QB8: now also J3.8 (Pin_8); no longer J3.9 (Pin_9)
- net RM: now also J2.4 (Pin_4); no longer J2.6 (Pin_6)
- net Rst1: now also J2.7 (Pin_7); no longer J2.3 (Pin_3)
- net Rst2: now also J3.9 (Pin_9); no longer J3.3 (Pin_3)
- net Rung2: now also J3.10 (Pin_10); no longer J3.11 (Pin_11)
- net Sin2: now also J3.11 (Pin_11); no longer J3.10 (Pin_10)
- net at C6.2, D4.1 (K), R5.2: now also U1.1; no longer U1.13
- net at C5.2, D3.1 (K), R4.2: now also U1.13; no longer U1.1
- new net: D3.2 (A), U1.11, U1.12
- new net: D4.2 (A), U1.2, U1.3
- no-connect marks 0 -> 7

Commit message: Updates to panel etc.
Parts:
- C4: renamed from C2; footprint Capacitor_THT:C_Radial_D5.0mm_H11.0mm_P2.00mm -> Capacitor_THT:C_Disc_D3.8mm_W2.6mm_P2.50mm
- C5: renamed from C3; footprint Capacitor_THT:C_Radial_D5.0mm_H11.0mm_P2.00mm -> Capacitor_THT:C_Disc_D3.8mm_W2.6mm_P2.50mm
- J21: renamed from J2; footprint Connector_PinSocket_2.54mm:PinSocket_1x12_P2.54mm_Vertical -> Connector_PinHeader_2.54mm:PinHeader_1x12_P2.54mm_Vertical
- J22: renamed from J3; footprint Connector_PinSocket_2.54mm:PinSocket_1x12_P2.54mm_Vertical -> Connector_PinHeader_2.54mm:PinHeader_1x12_P2.54mm_Vertical
- renumbered C8 to C10, C9 to C11, C10 to C12, C11 to C13, C12 to C14, C13 to C15, C1 to C3, C4 to C6, C5 to C7, C6 to C8, C7 to C9, D2 to D10, D3 to D11, D4 to D12, D1 to D9, J1 to J20, Q1 to Q10, Q2 to Q11, Q3 to Q12, Q4 to Q13, R36 to R34, R1 to R36, R2 to R37, R3 to R38, R4 to R39, R5 to R40, R6 to R41, R7 to R42, R8 to R43, R9 to R44, R10 to R45, R11 to R46, R12 to R47, R13 to R48, R14 to R49, R15 to R50, R16 to R51, R17 to R52, R18 to R53, R19 to R54, R20 to R55, R21 to R56, R22 to R57, R23 to R58, R24 to R59, R25 to R60, R26 to R61, R27 to R62, R28 to R63, R29 to R64, R30 to R65, R31 to R66, R32 to R67, R33 to R68, R34 to R69, U1 to U2, U2 to U3
Connections:
- net O1: now also U2.4; no longer U2.10
- net O2: now also U2.10; no longer U2.4
- net Rung1: now also U3.6 (-), U3.7; no longer U3.1, U3.2 (-)
- net Sin1: now also U3.1, U3.2 (-); no longer U3.6 (-), U3.7
- net at R62.2, R63.2, R64.2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: now also U3.5 (+); no longer U3.3 (+)
- net at C8.2, D12.1 (K), R40.2: now also U2.13; no longer U2.1
- net at R44.2, R45.2, R46.2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: now also U3.3 (+); no longer U3.5 (+)
- net at C7.2, D11.1 (K), R39.2: now also U2.1; no longer U2.13
- new net: D11.2 (A), U2.2, U2.3
- new net: D12.2 (A), U2.11, U2.12

Commit message: Removed the unneccessary 100ohm resistor after the expo converter
Parts:
- removed R39, R40: 100, Resistor_THT:R_Axial_DIN0204_L3.6mm_D1.6mm_P7.62mm_Horizontal, symbol Device:R
- C2: renamed from C4; footprint Capacitor_THT:C_Disc_D3.8mm_W2.6mm_P2.50mm -> Capacitor_THT:C_Radial_D5.0mm_H11.0mm_P2.00mm
- C3: renamed from C5; footprint Capacitor_THT:C_Disc_D3.8mm_W2.6mm_P2.50mm -> Capacitor_THT:C_Radial_D5.0mm_H11.0mm_P2.00mm
- J2: renamed from J21; footprint Connector_PinHeader_2.54mm:PinHeader_1x12_P2.54mm_Vertical -> Connector_PinSocket_2.54mm:PinSocket_1x12_P2.54mm_Vertical
- J3: renamed from J22; footprint Connector_PinHeader_2.54mm:PinHeader_1x12_P2.54mm_Vertical -> Connector_PinSocket_2.54mm:PinSocket_1x12_P2.54mm_Vertical
- renumbered C3 to C1, C12 to C10, C13 to C11, C14 to C12, C15 to C13, C6 to C4, C7 to C5, C8 to C6, C9 to C7, C10 to C8, C11 to C9, D9 to D1, D10 to D2, D11 to D3, D12 to D4, J20 to J1, Q10 to Q1, Q11 to Q2, Q12 to Q3, Q13 to Q4, R36 to R1, R45 to R10, R46 to R11, R47 to R12, R48 to R13, R49 to R14, R50 to R15, R51 to R16, R52 to R17, R53 to R18, R54 to R19, R37 to R2, R55 to R20, R56 to R21, R57 to R22, R58 to R23, R59 to R24, R60 to R25, R61 to R26, R62 to R27, R63 to R28, R64 to R29, R38 to R3, R65 to R30, R66 to R31, R67 to R32, R68 to R33, R69 to R34, R34 to R36, R41 to R6, R42 to R7, R43 to R8, R44 to R9, U2 to U1, U3 to U2
Connections:
- net O1: now also U1.10; no longer U1.4
- net O2: now also U1.4; no longer U1.10
- net Rung1: now also U2.1, U2.2 (-); no longer U2.6 (-), U2.7
- net Sin1: now also U2.6 (-), U2.7; no longer U2.1, U2.2 (-)
- net at R27.2, R28.2, R29.2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: now also U2.3 (+); no longer U2.5 (+)
- net at Q4.3 (C): now also C6.2, D4.1 (K), U1.1
- net at R10.2, R11.2, R12.2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: now also U2.5 (+); no longer U2.3 (+)
- net at Q3.3 (C): now also C5.2, D3.1 (K), U1.13
- new net: D3.2 (A), U1.11, U1.12
- new net: D4.2 (A), U1.2, U1.3

Commit message: Added negative CV protection diodes
Parts:
- C4: renamed from C2; footprint Capacitor_THT:C_Radial_D5.0mm_H11.0mm_P2.00mm -> Capacitor_THT:C_Disc_D3.8mm_W2.6mm_P2.50mm
- C5: renamed from C3; footprint Capacitor_THT:C_Radial_D5.0mm_H11.0mm_P2.00mm -> Capacitor_THT:C_Disc_D3.8mm_W2.6mm_P2.50mm
- J21: renamed from J2; footprint Connector_PinSocket_2.54mm:PinSocket_1x12_P2.54mm_Vertical -> Connector_PinHeader_2.54mm:PinHeader_1x12_P2.54mm_Vertical
- J22: renamed from J3; footprint Connector_PinSocket_2.54mm:PinSocket_1x12_P2.54mm_Vertical -> Connector_PinHeader_2.54mm:PinHeader_1x12_P2.54mm_Vertical
- renumbered C8 to C10, C9 to C11, C10 to C12, C11 to C13, C12 to C14, C13 to C15, C1 to C3, C4 to C6, C5 to C7, C6 to C8, C7 to C9, D2 to D10, D3 to D11, D4 to D12, D1 to D9, J1 to J20, Q1 to Q10, Q2 to Q11, Q3 to Q12, Q4 to Q13, R36 to R34, R1 to R36, R2 to R37, R3 to R38, R6 to R41, R7 to R42, R8 to R43, R9 to R44, R10 to R45, R11 to R46, R12 to R47, R13 to R48, R14 to R49, R15 to R50, R16 to R51, R17 to R52, R18 to R53, R19 to R54, R20 to R55, R21 to R56, R22 to R57, R23 to R58, R24 to R59, R25 to R60, R26 to R61, R27 to R62, R28 to R63, R29 to R64, R30 to R65, R31 to R66, R32 to R67, R33 to R68, R34 to R69, U1 to U2, U2 to U3
Connections:
- net O1: now also U2.4; no longer U2.10
- net O2: now also U2.10; no longer U2.4
- net Rung1: now also U3.6 (-), U3.7; no longer U3.1, U3.2 (-)
- net Sin1: now also U3.1, U3.2 (-); no longer U3.6 (-), U3.7
- net at R62.2, R63.2, R64.2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: now also U3.5 (+); no longer U3.3 (+)
- net at C8.2, D12.1 (K), Q13.3 (C): now also U2.13; no longer U2.1
- net at R44.2, R45.2, R46.2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: now also U3.3 (+); no longer U3.5 (+)
- net at C7.2, D11.1 (K), Q12.3 (C): now also U2.1; no longer U2.13
- new net: D11.2 (A), U2.2, U2.3
- new net: D12.2 (A), U2.11, U2.12

Commit message: Added range switch
Parts:
- removed C7: 10nF, Capacitor_THT:C_Disc_D5.0mm_W2.5mm_P2.50mm, symbol Device:C
- removed C8: 10nf, Capacitor_THT:C_Disc_D5.0mm_W2.5mm_P2.50mm, symbol Device:C
Connections:
- net Clk2: now also J22.8 (Pin_8); no longer J22.7 (Pin_7)
- net D2: now also J22.5 (Pin_5); no longer J22.4 (Pin_4)
- net GND: no longer J22.12 (Pin_12)
- net Osc2: now also J22.6 (Pin_6); no longer J22.5 (Pin_5)
- net Osc3: now also J22.7 (Pin_7); no longer J22.6 (Pin_6)
- net Osc3sw: now also J22.4 (Pin_4); no longer J22.3 (Pin_3)
- net QB8: now also J22.9 (Pin_9); no longer J22.8 (Pin_8)
- net Rst2: now also J22.10 (Pin_10); no longer J22.9 (Pin_9)
- net Rung2: now also J22.11 (Pin_11); no longer J22.10 (Pin_10)
- net Sin2: now also J22.12 (Pin_12); no longer J22.11 (Pin_11)
- net RATESEL2: now reaches D12.1 (K), Q13.3 (C), U2.13
- net RATESEL2: now also J22.3 (Pin_3)
- net RATESEL1: now reaches D11.1 (K), Q12.3 (C), U2.1
- net RATESEL1: now also J21.3 (Pin_3)
- no-connect marks 7 -> 6
